File: SmallBuck/SmallBuck.kicad_sch (KiCad schematic)
At the start: 15 parts, among them J1 IN, J2 OUT, J3 OUT, J4 OUT, J5 OUT, U1 LMR51430

Commit message: ok
Parts:
- removed J5: OUT, Connector_JST:JST_XH_B2B-XH-A_1x02_P2.50mm_Vertical, symbol Connector:Conn_01x02_Socket
- added C7: 100-470uF, Capacitor_THT:CP_Radial_D8.0mm_P3.50mm, symbol Device:C_Polarized
- added H1, H2, H3, H4: MountingHole, MountingHole:MountingHole_4mm, symbol Mechanical:MountingHole
Connections:
- net 5V: now also C7.1
- net GND: now also C7.2
Other:
- moved on the sheet: C5
